File: proves-prime-mainboard-v1/Connectors.kicad_sch (KiCad schematic)
At the start: 0 parts

Commit message: Migrated FC Board Elements
Parts:
- added H1, H2: MountingHole, symbol Mechanical:MountingHole
- added J3: Conn_ARM_JTAG_SWD_10, FC_DEV_BOARD:JTAG_2X05_1.27MM_BOX_NOCREAM, symbol Connector:Conn_ARM_JTAG_SWD_10
- added J4: BM04B-SRSS-TB(LF)(SN), FC_DEV_BOARD:JST_BM04B-SRSS-TB(LF)(SN), symbol BM04B-SRSS-TB_LF__SN_:BM04B-SRSS-TB(LF)(SN)
- added J5: USB_B_Micro, FC_DEV_BOARD:MOLEX_105164-0001, symbol Connector:USB_B_Micro
- added R26, R27: 22, Resistor_SMD:R_0603_1608Metric, symbol mainboard:RESISTOR0603
Connections:
- new net +3V3: J3.1 (VTref)
- new net D+: R26.1
- new net D-: R27.1
- new net GND: J3.3 (GND), J3.5 (GND), J3.9 (GNDDetect), J4.4, J4.S1 (SHIELD), J4.S2 (SHIELD), J5.5 (GND), J5.SH1 (Shield)
- new net SWCLK: J3.4 (SWDCLK/TCK)
- new net SWDIO: J3.2 (SWDIO/TMS)
- new net USB_D+: J4.3, J5.3 (D+), R26.2
- new net USB_D-: J4.2, J5.2 (D-), R27.2
- new net VBUS: J4.1, J5.1 (VBUS)
- new net ~{RESET}: J3.10 (~{RESET})
- no-connect marks 0 -> 3
Other:
- note added: "MOLEX_105164-0001"

Commit message: Migrated Power Monitor ICs
Changed lines of the file:
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@@
 		(on_board yes)
 		(dnp no)
-		(fields_autoplaced yes)
 		(property "Reference" "J4"
-			(at 90.805 35.56 0)
+			(at 82.55 25.908 0)
 			(effects
 				(font
@@
 		)
 		(property "Value" "BM04B-SRSS-TB(LF)(SN)"
-			(at 90.805 38.1 0)
+			(at 71.628 49.276 0)
 			(effects
 				(font

Commit message: Added Voltage Regulators
LT8610 3v3 and 5v

Co-Authored-By: rrakushkin <128992626+rrakushkin@users.noreply.github.com>
Changed lines of the file:
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@@
 	(text "MOLEX_105164-0001"
 		(exclude_from_sim no)
-		(at 21.59 46.99 90)
+		(at 20.32 45.974 90)
 		(effects
 			(font
@@
 		)
 		(property "Value" "22"
-			(at 50.546 31.9532 0)
+			(at 46.228 28.448 0)
 			(effects
 				(font
@@
 		)
 		(property "Value" "22"
-			(at 50.6476 39.9796 0)
-			(effects
-				(font
+			(at 46.736 41.656 0)
+			(effects
+				(font

Commit message: Added USB-C Connector
Parts:
- J4: footprint FC_DEV_BOARD:JST_BM04B-SRSS-TB(LF)(SN) -> FC_DEV_BOARD:JST_BM04B-SRSS-TB(LF)(SN)
Changed lines of the file:
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@@
 			)
 		)
-		(property "Footprint" "FC_DEV_BOARD:JST_BM04B-SRSS-TB(LF)(SN) "
+		(property "Footprint" "FC_DEV_BOARD:JST_BM04B-SRSS-TB(LF)(SN)"
 			(at 83.82 38.1 0)
 			(effects

Commit message: More Wiring!
Connected Additional Peripheral
Parts:
- removed J5: USB_B_Micro, FC_DEV_BOARD:MOLEX_105164-0001, symbol Connector:USB_B_Micro
- removed R26, R27: 22, Resistor_SMD:R_0603_1608Metric, symbol mainboard:RESISTOR0603
Connections:
- no-connect marks 3 -> 2
Other:
- note added: "Auxilery USB"
- note removed: "MOLEX_105164-0001"
- moved on the sheet: J4
