File: proves-prime-mainboard-v1/eps_pms.kicad_sch (KiCad schematic)
At the start: 0 parts

Commit message: Migrated Power Monitor ICs
Parts:
- added C39, C41: 10uF, Capacitor_SMD:C_0603_1608Metric, symbol mainboard:10UF-0603-6.3V-20%
- added C40: 1uF, Capacitor_SMD:C_0603_1608Metric, symbol mainboard:10UF-0603-6.3V-20%
- added C42, C43: 0.1uF, Capacitor_SMD:C_0603_1608Metric, symbol Device:C_Small
- added D10, D11, D12, D14: DFLS130L-7, Diode_SMD:D_PowerDI-123, symbol Device:D_Schottky
- added D13, D15: DFLS130L, Diode_SMD:D_PowerDI-123, symbol Device:D_Schottky
- added IC4: LT3652IMSE#PBF, Package_SO:MSOP-12-1EP_3x4mm_P0.65mm_EP1.65x2.85mm, symbol LT3652IMSE#PBF:LT3652IMSE#PBF
- added L1: 10uH, Inductor_SMD:L_1812_4532Metric, symbol Device:L
- added R40: 100K, Resistor_SMD:R_0603_1608Metric, symbol Device:R_US
- added R41: 100k, Resistor_SMD:R_0603_1608Metric, symbol mainboard:R-US_R0603
- added R42: 94k, Resistor_SMD:R_0603_1608Metric, symbol mainboard:R-US_R0603
- added R43: 10K, Resistor_SMD:R_0603_1608Metric, symbol Device:R_US
- added R44: 634k, Resistor_SMD:R_0603_1608Metric, symbol mainboard:R-US_R0603
- added R45: 412k, Resistor_SMD:R_0603_1608Metric, symbol mainboard:R-US_R0603
- added R46: 0.1, Resistor_SMD:R_2512_6332Metric, symbol mainboard:R-US_R0603
- added R47, R48: 0.002, Resistor_SMD:R_2512_6332Metric, symbol mainboard:R-US_R2512
- added U12, U13: INA219AxD, Package_SO:SOIC-8_3.9x4.9mm_P1.27mm, symbol Analog_ADC:INA219AxD
Connections:
- new net: C40.1, D14.1 (K), IC4.12 (SW), L1.1
- new net: IC4.10 (SENSE), L1.2, R46.2
- new net: IC4.7 (VFB), R44.1, R45.2
- new net: C39.1, D10.1 (K), D11.1 (K), IC4.1 (VIN), IC4.3 (~{SHDN}), R40.1
- new net: C40.2, D13.1 (K), IC4.11 (BOOST)
- new net: IC4.2 (VIN_REG), R41.2, R42.2
- new net: R40.2, R41.1
- new net +3V3: C42.2, C43.2, R43.1, U12.1 (A1), U12.5 (VS), U13.5 (VS)
- new net CHRG': IC4.4 (~{CHRG}), R43.2
- new net Dir_Chrg_In: D11.2 (A), D12.2 (A)
- new net GND: C39.2, C41.2, C42.1, C43.1, D14.2 (A), IC4.13 (EP), IC4.6 (TIMER), R42.1, R45.1, U12.2 (A0), U12.6 (GND), U13.1 (A1), U13.2 (A0), U13.6 (GND)
- new net PACK+: R48.2, U13.8 (IN+)
- new net SCL0: U12.4 (SCL), U13.4 (SCL)
- new net SDA0: U12.3 (SDA), U13.3 (SDA)
- new net VBATT_SENSE: C41.1, D13.2 (A), D15.2 (A), IC4.9 (BAT), R44.2, R46.1, R48.1, U13.7 (IN-)
- new net VBatt: D12.1 (K), D15.1 (K)
- new net VSOLAR: R47.2, U12.8 (IN+)
- new net VSOLAR_I: D10.2 (A), R47.1, U12.7 (IN-)
- no-connect marks 0 -> 2
Other:
- note added: "2S Li-Ion Battery Solar Charging Circuit"
- note added: "Battery Power Monitor 0x40"
- note added: "Current Sense Resistor: 2mOhm suggested on datasheet"
- note added: "Schottky Diode"
- note added: "Solar Power Monitor 0x41"
- note added: "VSOLAR 9V to 40V"

Commit message: Added Voltage Regulators
LT8610 3v3 and 5v

Co-Authored-By: rrakushkin <128992626+rrakushkin@users.noreply.github.com>
Other:
- moved on the sheet: C43, R48, U13

Commit message: More Wiring!
Connected Additional Peripheral
Connections:
- net CHRG' renamed ~{CHARGE}
Changed lines of the file:
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@@
+	)
+	(junction
+		(at 68.58 72.39)
+		(diameter 0)
+		(color 0 0 0 0)
 	)
 	(junction
@@
 	(wire
 		(pts
+			(xy 68.58 62.23) (xy 68.58 72.39)
+		)
+		(stroke
+			(width 0)
+			(type default)
+		)
+	)
+	(wire
+		(pts
 			(xy 109.22 52.07) (xy 109.22 53.34)
 		)
@@
 	(wire
 		(pts
-			(xy 68.58 62.23) (xy 68.58 72.39)
-		)
-		(stroke
-			(width 0)
-			(type default)
-		)
-	)
-	(wire
-		(pts
 			(xy 81.28 139.7) (xy 81.28 138.43)
 		)
@@
 		(pts
 			(xy 101.6 133.35) (xy 106.68 133.35)
+		)
+		(stroke
+			(width 0)
+			(type default)
+		)
+	)
+	(wire
+		(pts
+			(xy 67.31 72.39) (xy 68.58 72.39)
 		)
 		(stroke
@@
 		)
 	)
-	(global_label "CHRG'"
-		(shape input)
-		(at 68.58 72.39 180)
+	(global_label "~{CHARGE}"
+		(shape output)
+		(at 67.31 72.39 180)
 		(fields_autoplaced yes)
 		(effects
@@
 		)
 		(property "Intersheetrefs" "${INTERSHEET_REFS}"
-			(at 60.4217 72.3106 0)
+			(at 56.9467 72.39 0)
 			(effects
 				(font
