File: proves-prime-mainboard-v1/radios.kicad_sch (KiCad schematic)
At the start: 0 parts

Commit message: Migrated FC Board Elements
Parts:
- added C36: 10uF, Capacitor_SMD:C_0603_1608Metric, symbol Device:C_Small
- added J9: Conn_Coaxial, Connector_Coaxial:SMA_Amphenol_901-144_Vertical, symbol Connector:Conn_Coaxial
- added JP5: Jumper_3_Open, Jumper:SolderJumper-3_P1.3mm_Open_RoundedPad1.0x1.5mm_NumberLabels, symbol Jumper:Jumper_3_Open
- added R37: 10k, Resistor_SMD:R_0603_1608Metric, symbol mainboard:10KOHM-1_10W-1%(0603)0603
- added U7: RFM98PW, FC_DEV_BOARD:RFM98PW, symbol mainboard:RFM98PW
- added U8: RFM9xBreakout, RF_Module:HOPERF_RFM9XW_SMD, symbol mainboard:RFM9xBreakout
Connections:
- new net +3V3: JP5.1 (A), R37.1, U7.9 (3.3V)
- new net GND: C36.1, J9.2 (Ext), U7.16 (GND), U7.17 (GND), U7.2 (GND), U8.1 (GND), U8.10 (GND), U8.8 (GND)
- new net RF1_ANT: J9.1 (In), U7.1 (ANT), U8.9 (ANT)
- new net RF1_IO0: U7.6 (GPIO_0), U8.14 (DIO0)
- new net RF1_IO4: U7.4 (GPIO_4), U8.12 (BUSY)
- new net RF1_RST: U7.14 (RESET), U8.6 (~{RESET})
- new net RF_VCC: C36.2, JP5.2 (C), U7.5 (VCC), U8.13 (3V3)
- new net SPI0_CS0: R37.2, U7.13 (NSS), U8.5 (CS)
- new net SPI0_MISO: U7.10 (MISO), U8.2 (MISO)
- new net SPI0_MOSI: U7.11 (MOSI), U8.3 (MOSI)
- new net SPI0_SCK: U7.12 (SCK), U8.4 (SCK)
- new net VCC_RF1: JP5.3 (B)
- no-connect marks 0 -> 8
Other:
- note added: "Modular Radios (HopeRF format)"
- note added: "Radio #1"

Commit message: Duplicated Radios
Parts:
- added C37: 10uF, Capacitor_SMD:C_0603_1608Metric, symbol Device:C_Small
- added J10: Conn_Coaxial, Connector_Coaxial:SMA_Amphenol_901-144_Vertical, symbol Connector:Conn_Coaxial
- added JP6: Jumper_3_Open, Jumper:SolderJumper-3_P1.3mm_Open_RoundedPad1.0x1.5mm_NumberLabels, symbol Jumper:Jumper_3_Open
- added R39: 10k, Resistor_SMD:R_0603_1608Metric, symbol mainboard:10KOHM-1_10W-1%(0603)0603
- added U10: RFM9xBreakout, RF_Module:HOPERF_RFM9XW_SMD, symbol mainboard:RFM9xBreakout
- added U9: RFM98PW, FC_DEV_BOARD:RFM98PW, symbol mainboard:RFM98PW
Connections:
- net +3V3: now also JP6.1 (A), R39.1, U9.9 (3.3V)
- net GND: now also C37.1, J10.2 (Ext), U10.1 (GND), U10.10 (GND), U10.8 (GND), U9.16 (GND), U9.17 (GND), U9.2 (GND)
- net SPI0_CS0: now also R39.2, U10.5 (CS), U9.13 (NSS)
- net VCC_RF1: now also JP6.3 (B)
- net RF_VCC renamed RF1_VCC
- new net RF2_ANT: J10.1 (In), U10.9 (ANT), U9.1 (ANT)
- new net RF2_IO0: U10.14 (DIO0), U9.6 (GPIO_0)
- new net RF2_IO4: U10.12 (BUSY), U9.4 (GPIO_4)
- new net RF2_RST: U10.6 (~{RESET}), U9.14 (RESET)
- new net RF2_VCC: C37.2, JP6.2 (C), U10.13 (3V3), U9.5 (VCC)
- no-connect marks 8 -> 16
Other:
- note added: "Radio #2 (Auxilery)"
- moved on the sheet: R37

Commit message: Removed Unneeded Stuff
- Took away small RFM footprint from Radio 1
- Removed the cursed CAN bus
Parts:
- removed U8: RFM9xBreakout, RF_Module:HOPERF_RFM9XW_SMD, symbol mainboard:RFM9xBreakout
Connections:
- no-connect marks 16 -> 12
Other:
- moved on the sheet: C37, J10, JP5, JP6, R39, U10, U9

Commit message: More Wiring!
Connected Additional Peripheral
Connections:
- net SPI0_CS0: no longer R39.2, U10.5 (CS), U9.13 (NSS)
- new net: R39.2, U10.5 (CS), U9.13 (NSS)
Changed lines of the file:
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@@
-	(wire
-		(pts
-			(xy 26.67 91.44) (xy 29.21 91.44)
-		)
-		(stroke
-			(width 0)
-			(type default)
-		)
-	)
 	(wire
 		(pts
@@
 				(hide yes)
 			)
-		)
-	)
-	(global_label "SPI0_CS0"
-		(shape bidirectional)
-		(at 26.67 91.44 180)
-		(fields_autoplaced yes)
-		(effects
-			(font
-				(size 1.27 1.27)
-			)
-			(justify right)
-		)
-		(property "Intersheetrefs" "${INTERSHEET_REFS}"
-			(at 13.7025 91.44 0)
-			(effects
-				(font
-					(size 1.27 1.27)
-				)
-				(justify right)
-				(hide yes)
-			)
