File: proves-prime-mainboard-v1/burn_heat.kicad_sch (KiCad schematic)
At the start: 0 parts

Commit message: Added Burnwire Candidates
Parts:
- added D7: DFLS130L, Diode_SMD:D_PowerDI-123, symbol Device:D_Schottky
- added D8: 1N4151WS, Diode_SMD:D_SOD-323, symbol oresat-diodes:1N4151WS-HE3
- added K1: APAN3105, APAN3105:RELAY_APAN3105, symbol APAN3105:APAN3105
- added Q1: MMBT2222AT, Package_TO_SOT_SMD:SOT-523, symbol mainboard:MMBT2222AT
- added Q2, Q3: IRLML2803, Package_TO_SOT_SMD:SOT-23, symbol mainboard:IRLML2803TRPBF
- added Q4, Q5: NDS8434, Package_SO:SOIC-8-1EP_3.9x4.9mm_P1.27mm_EP2.514x3.2mm, symbol mainboard:NDS8434
- added Q6: FDMQ86530L, oresat-transistors:FDMQ86530L, symbol oresat-transistors:FDMQ86530L
- added Q7, Q8: DMP2240UDM-7, Package_TO_SOT_SMD:SOT-23-6, symbol oresat-transistors:DMP2240UDM-7
- added R56, R59, R60: 10k, Resistor_SMD:R_0603_1608Metric, symbol mainboard:RESISTOR0603
- added R57: 100, Resistor_SMD:R_0603_1608Metric, symbol mainboard:RESISTOR0603
- added R58: 634k, Resistor_SMD:R_0603_1608Metric, symbol mainboard:R-US_R0603
- added R61, R62: 4.7k, Resistor_SMD:R_0603_1608Metric, symbol mainboard:RESISTOR0603
- added R63, R64: 100k, Resistor_SMD:R_0603_1608Metric, symbol mainboard:RESISTOR0603
- added R65, R66, R67, R70: 10k, Resistor_SMD:R_0603_1608Metric, symbol Device:R_Small_US
- added R68: 1k, Resistor_SMD:R_0603_1608Metric, symbol Device:R_Small_US
- added R69: 47k, Resistor_SMD:R_0603_1608Metric, symbol Device:R_Small_US
- added TP13, TP14, TP15, TP9: Test-Point, oresat-misc:TestPoint_Pad_D1.0mm, symbol oresat-misc:Test-Point-1mm-round
Connections:
- new net: D7.2 (A), K1.C2, Q1.3 (C)
- new net: K1.NO, Q4.1 (Source), Q4.2 (Source), Q4.3 (Source), Q5.1 (Source), Q5.2 (Source), Q5.3 (Source), R58.2, R63.2, R64.2
- new net: Q1.2 (E), R57.1
- new net: Q8.2 (S), Q8.6 (D)
- new net: Q6.11 (D1/D4), Q6.13 (D1/D4), Q6.2 (D1/D4), Q7.1 (G), Q7.3 (G), Q8.1 (G), Q8.3 (G), R67.2
- new net: Q2.1 (G), R61.1
- new net: Q3.1 (G), R62.1
- new net: D8.2, R68.2
- new net: Q3.3 (D), Q5.4 (Gate), R64.1
- new net: Q7.2 (S), Q7.6 (D)
- new net: Q2.3 (D), Q4.4 (Gate), R63.1
- new net BURN_RELAY_A: Q1.1 (B), R56.1
- new net DEPLOY_ANTENNAS: D8.1, Q7.4 (D), Q8.4 (D), R69.1, TP15.1
- new net ENAB_BURN: R60.1, R62.2
- new net ENAB_HEATER: R59.1, R61.2
- new net FIRE_ANTENNAS_1: Q6.1 (G1), Q6.9 (G3), R66.1, TP9.1
- new net FIRE_ANTENNAS_2: Q6.12 (G4), Q6.4 (G2), R65.1, TP13.1
- new net GND: Q2.2 (S), Q3.2 (S), Q4.5 (Drain), Q4.6 (Drain), Q4.7 (Drain), Q4.8 (Drain), Q5.5 (Drain), Q5.6 (Drain), Q5.7 (Drain), Q5.8 (Drain), Q6.5 (S2), Q6.6 (S2), Q6.7 (S3), Q6.8 (S3), R56.2, R57.2, R58.1, R59.2, R60.2, R65.2, R66.2, R70.2
- new net PACK+: K1.M
- new net READ_ANTENNAS: R69.2, R70.1, TP14.1
- new net TEST_ANTENNAS: R68.1
- new net VBUS: Q7.5 (S), Q8.5 (S), R67.1
- new net VBUSP: D7.1 (K), K1.C1
- no-connect marks 0 -> 4
Other:
- note added: "(6.0, 7.2, 8.4)V"
- note added: "Burn Wire Control (Antenna Depolyment) OreSat Based System"
- note added: "Burn Wire Control (Antenna Depolyment) PyCubed Based System"
- note added: "Must not go above 1.8V for Octavo ADC"
- note added: "Power Relay A"

Commit message: Created MVS Sheet
Minimum Viable Satellite
Connections:
- net DEPLOY_ANTENNAS renamed DEPLOY1
- net FIRE_ANTENNAS_1 renamed FIRE_DEPLOY1_A
- net FIRE_ANTENNAS_2 renamed FIRE_DEPLOY1_B
- net READ_ANTENNAS renamed READ_DEPLOY1
Changed lines of the file:
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@@
 		)
 	)
-	(global_label "FIRE_ANTENNAS_1"
+	(global_label "FIRE_DEPLOY1_A"
 		(shape input)
 		(at 34.29 157.48 180)
@@
 		)
 		(property "Intersheetrefs" "${INTERSHEET_REFS}"
-			(at 14.6323 157.48 0)
-			(effects
-				(font
-					(size 1.27 1.27)
-				)
-				(justify right)
-				(hide yes)
-			)
-		)
-	)
-	(global_label "FIRE_ANTENNAS_2"
+			(at 15.8229 157.48 0)
+			(effects
+				(font
+					(size 1.27 1.27)
+				)
+				(justify right)
+				(hide yes)
+			)
+		)
+	)
+	(global_label "FIRE_DEPLOY1_B"
 		(shape input)
 		(at 34.29 161.29 180)
@@
 		)
 		(property "Intersheetrefs" "${INTERSHEET_REFS}"
-			(at 14.6323 161.29 0)
+			(at 15.6415 161.29 0)
 			(effects
 				(font
@@
 		)
 	)
-	(global_label "DEPLOY_ANTENNAS"
+	(global_label "DEPLOY1"
 		(shape output)
 		(at 158.75 152.4 0)
@@
 		)
 		(property "Intersheetrefs" "${INTERSHEET_REFS}"
-			(at 179.2544 152.4 0)
+			(at 170.0809 152.4 0)
 			(effects
 				(font
@@
 		)
 	)
-	(global_label "READ_ANTENNAS"
+	(global_label "READ_DEPLOY1"
 		(shape output)
 		(at 116.84 168.91 180)
@@
 		)
 		(property "Intersheetrefs" "${INTERSHEET_REFS}"
-			(at 98.6942 168.91 0)
-			(effects
-				(font
+			(at 99.7639 168.91 0)
+			(effects
+				(font
