File: proves-prime-mainboard-v1/watchdog.kicad_sch (KiCad schematic)
At the start: 40 parts, among them J1 Breakout, J2 Breakout, U2 TLV1704

Commit message: Created MVS Sheet
Minimum Viable Satellite
Connections:
- net WDT_WDI renamed RP2350_WDT_WDI
Changed lines of the file:
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@@
 		)
 	)
-	(global_label "WDT_WDI"
+	(global_label "RP2350_WDT_WDI"
 		(shape input)
 		(at 83.82 124.46 180)
@@
 		)
 		(property "Intersheetrefs" "${INTERSHEET_REFS}"
-			(at 72.376 124.46 0)
+			(at 64.0304 124.46 0)
 			(effects
 				(font
